File: RCT-X-Telemetry.kicad_pcb (KiCad board)
At the start: 2 copper layers, 30 x 70 mm, 83 parts, among them J1 USB_B_Micro, J2 USB_B_Micro, P1 KRC_Conn_SWD, Q1 Q_NMOS_DGS, U1 KRC_Conn_CAN, U2 LT1761-5, U3 LT1965xDD-3.3, U4 NCV7342, U5 CY8C58xxLTI-LPxxx, U6 FT234XD, U7 RM-92X, U8 W25N01GVxxIG-IT, Y1 Crystal_kHz, Y2 Crystal_MHz

Commit message: Completed Rev2
Parts:
- removed C26, C27: 0.1uF, Capacitor_SMD:C_0402_1005Metric
- removed D2: LED_ORANGE, LED_SMD:LED_0603_1608Metric
- removed G***: LOGO, KUTKiCad_footprint:yuru
- removed G***: LOGO, KUTKiCad_footprint:logo
- removed Y2: Crystal_MHz, KUTKiCad_footprint:Crystal_Murata_XRCHA
- added F1: Polyfuse, Fuse:Fuse_0805_2012Metric, B.Cu at (57.2, 76.7)
- added R34: 1kΩ, Resistor_SMD:R_0402_1005Metric, B.Cu at (54.4, 112.0)
- C21, C23: value 9pF -> 0.1uF; footprint Capacitor_SMD:C_0201_0603Metric -> Capacitor_SMD:C_0402_1005Metric
- C22: value 0.1uF -> 10uF; footprint Capacitor_SMD:C_0402_1005Metric -> Capacitor_SMD:C_0603_1608Metric
- C24: value 10uF -> 0.1uF; footprint Capacitor_SMD:C_0603_1608Metric -> Capacitor_SMD:C_0402_1005Metric
- D1: value LED_BLUE -> LED_RGBA; footprint LED_SMD:LED_0603_1608Metric -> KUTKiCad_footprint:LED_LiteOn_LTST-C19HE1WT
- H1, H2, H3, H4: footprint MountingHole:MountingHole_3.5mm -> MountingHole:MountingHole_3.2mm_M3
- R13: value 22Ω -> 47kΩ
- R18: value 22Ω -> 4.7kΩ
- R20: value 4.7kΩ -> 47kΩ
- R29: value 47kΩ -> 22Ω
- R3: value 1MΩ -> 22Ω; moved to F.Cu
- R30: value 4.7kΩ -> 22Ω
- R32: value 1kΩ -> 4.7kΩ
- R5: value 22Ω -> 1.5kΩ
- R6, R7: value R -> 820Ω
- R8: value 47kΩ -> 1MΩ; moved to F.Cu
- TH1: moved to F.Cu
- U6: value FT234XD -> RM-92X; footprint Package_DFN_QFN:DFN-12-1EP_3x3mm_P0.45mm_EP1.66x2.38mm -> KUTKiCad_footprint:RFLink_Module_RM-92A; moved to F.Cu
- U7: value RM-92X -> FT234XD; footprint KUTKiCad_footprint:RFLink_Module_RM-92A -> Package_DFN_QFN:DFN-12-1EP_3x3mm_P0.45mm_EP1.66x2.38mm; moved to B.Cu
- Y1: value Crystal_kHz -> Crystal_MHz; footprint KUTKiCad_footprint:Crystal_SeikoEpson_FC-135 -> KUTKiCad_footprint:Crystal_Murata_XRCHA
- moved R18 35.6 mm to (41.1, 81.1), turned to 270 degrees
- moved C25 34.1 mm to (41.1, 78.9)
- moved R30 34.0 mm to (48.2, 115.9), turned to 0 degrees
- moved R32 28.5 mm to (53.1, 83.5), turned to 90 degrees
- moved R17 27.7 mm to (50.3, 87.1), turned to 315 degrees
- moved R20 24.2 mm to (65.5, 103.6), turned to 0 degrees
- moved C21 23.3 mm to (51.1, 111.0), turned to 90 degrees
- moved C23 23.2 mm to (53.9, 110.5), turned to 90 degrees
- moved R13 22.6 mm to (46.5, 110.0), turned to 180 degrees
- moved R25 19.1 mm to (46.5, 99.8)
- moved U6 16.4 mm to (67.5, 112.5), turned to 180 degrees
- moved U7 16.4 mm to (51.4, 115.3), turned to 270 degrees
- moved TH1 15.9 mm to (50.0, 88.0), turned to 180 degrees
- moved R8 15.8 mm to (50.0, 89.5), turned to 0 degrees
- moved R29 11.3 mm to (48.2, 114.8)
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Connections:
- C23 pad 1: Net-(C23-Pad1) -> Net-(C22-Pad1)
- C24 pad 1: Net-(C24-Pad1) -> /FTDI-~RESET
- C25 pad 1: Net-(C24-Pad1) -> +3V3
- J2 pad 1: Net-(C24-Pad1) -> Net-(C22-Pad1)
- R13 pad 2: /Flash-MISO -> +3V3
- R14 pad 2: /Flash-MOSI -> /Flash-MISO
- R15 pad 2: /Flash-SCLK -> /Flash-MOSI
- R16 pad 2: /Flash-~CS -> /Flash-SCLK
- R17 pad 1: Net-(J2-Pad3) -> Net-(R17-Pad1)
- R17 pad 2: Net-(R17-Pad2) -> /Flash-~CS
- R18 pad 1: Net-(J2-Pad2) -> +3V3
- R29 pad 1: +3V3 -> Net-(J2-Pad3)
- R3 pad 1: Net-(R3-Pad1) -> Net-(J1-Pad3)
- R3 pad 2: GND -> Net-(R3-Pad2)
- R30 pad 1: +3V3 -> Net-(J2-Pad2)
- R30 pad 2: Net-(R16-Pad1) -> Net-(R30-Pad2)
- R31 pad 2: Net-(R13-Pad1) -> Net-(R17-Pad1)
- R32 pad 1: Net-(C24-Pad1) -> +3V3
- R32 pad 2: /FTDI-~RESET -> Net-(R14-Pad1)
- R4 pad 1: Net-(J1-Pad3) -> Net-(J1-Pad2)
- R5 pad 1: Net-(J1-Pad2) -> Net-(D1-Pad1)
- R6 pad 1: +3V3 -> Net-(D1-Pad2)
- R6 pad 2: Net-(D1-Pad2) -> Net-(R6-Pad2)
- R7 pad 1: +3V3 -> Net-(D1-Pad3)
- R7 pad 2: Net-(D2-Pad2) -> Net-(R7-Pad2)
- R8 pad 2: +3V3 -> GND
- TH1 pad 2: Net-(R3-Pad1) -> Net-(R8-Pad1)
- U1 pad 2: Net-(C1-Pad1) -> Net-(F1-Pad2)
- U5 pad 22: Net-(R4-Pad2) -> Net-(R3-Pad2)
- U5 pad 23: Net-(R5-Pad2) -> Net-(R4-Pad2)
- U5 pad 27: Net-(C23-Pad1) -> Net-(C20-Pad1)
- U5 pad 28: Net-(C21-Pad1) -> Net-(C19-Pad1)
- U5 pad 32: Net-(R3-Pad1) -> Net-(R5-Pad2)
- U5 pad 33: Net-(D1-Pad1) -> Net-(R6-Pad2)
- U5 pad 34: Net-(D2-Pad1) -> Net-(R7-Pad2)
- U5 pad 4: Net-(U5-Pad4) -> Net-(R8-Pad1)
- U5 pad 40: Net-(C20-Pad1) -> Net-(U5-Pad40)
- U5 pad 41: Net-(C19-Pad1) -> Net-(U5-Pad41)
- U6 pad 1: Net-(R17-Pad2) -> GND
- U6 pad 10: /FTDI-RXD -> Net-(R21-Pad2)
- U6 pad 11: Net-(U6-Pad11) -> Net-(R23-Pad2)
- U6 pad 12: Net-(R18-Pad2) -> Net-(R24-Pad2)
- U6 pad 13: GND -> /Radio-TXD
- U6 pad 2: /FTDI-~RESET -> /Radio-~RESET
- U6 pad 3: Net-(C22-Pad1) -> Net-(Q1-Pad3)
- U6 pad 4: Net-(C24-Pad1) -> Net-(U6-Pad4)
- U6 pad 5: GND -> Net-(R22-Pad2)
- U6 pad 6: Net-(U6-Pad6) -> /Radio-CTS
- U6 pad 7: /FTDI-TXD -> /Radio-RTS
- U6 pad 8: Net-(U6-Pad8) -> Net-(R20-Pad2)
- U6 pad 9: Net-(C22-Pad1) -> Net-(U6-Pad9)
- U7 pad 1: GND -> Net-(R29-Pad2)
- U7 pad 10: Net-(R22-Pad2) -> /FTDI-RXD
- U7 pad 11: Net-(R24-Pad2) -> Net-(U7-Pad11)
- U7 pad 12: Net-(R25-Pad2) -> Net-(R30-Pad2)
- U7 pad 13: /Radio-TXD -> GND
- U7 pad 2: /Radio-~RESET -> /FTDI-~RESET
- U7 pad 3: Net-(Q1-Pad3) -> Net-(C21-Pad1)
- U7 pad 4: Net-(U7-Pad4) -> Net-(C22-Pad1)
- U7 pad 5: Net-(R23-Pad2) -> GND
- U7 pad 6: /Radio-CTS -> Net-(U7-Pad6)
- U7 pad 7: /Radio-RTS -> /FTDI-TXD
- U7 pad 8: Net-(R21-Pad2) -> Net-(U7-Pad8)
- U7 pad 9: Net-(U7-Pad9) -> Net-(C21-Pad1)
- U8 pad 1: Net-(R16-Pad1) -> Net-(R17-Pad1)
- U8 pad 2: Net-(R13-Pad1) -> Net-(R14-Pad1)
- U8 pad 3: Net-(R20-Pad2) -> Net-(R19-Pad2)
- U8 pad 5: Net-(R14-Pad1) -> Net-(R15-Pad1)
- U8 pad 6: Net-(R15-Pad1) -> Net-(R16-Pad1)
- U8 pad 7: Net-(R19-Pad2) -> Net-(R18-Pad2)
Routing:
- net GND: track 33.4 -> 2.23 mm, vias 81 -> 94
- net Net-(C24-Pad1): track 21.7 -> 0.00 mm, vias 2 -> 0
- net +3V3: track 184.7 -> 202.9 mm, vias 13 -> 11
- net Net-(R17-Pad1): track 0.00 -> 16.1 mm
- net Net-(C22-Pad1): track 9.12 -> 21.8 mm
- net Net-(R3-Pad2): track 0.00 -> 12.6 mm, vias 0 -> 1
- net Net-(R3-Pad1): track 12.0 -> 0.00 mm
- net Net-(D2-Pad1): track 10.4 -> 0.00 mm, vias 1 -> 0
- net Net-(D1-Pad1): track 11.2 -> 1.68 mm, vias 1 -> 0
- net Net-(R13-Pad1): track 10.9 -> 1.47 mm
- net Net-(R6-Pad2): track 0.00 -> 8.84 mm, vias 0 -> 1
- net Net-(C1-Pad1): track 32.6 -> 40.6 mm, vias 0 -> 2
- net Net-(R7-Pad2): track 0.00 -> 7.48 mm, vias 0 -> 1
- net /Flash-MOSI: track 3.79 -> 10.4 mm
- net Net-(C21-Pad1): track 6.09 -> 12.6 mm, vias 0 -> 2
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Other:
- board text added: "12[5] : Themistor"
- board text added: "3[3] : LED-RED 3[4] : LED-GREEN 3[5] : LED-BLUE"
- board text added: "v2"
- board text removed: "3[3] : Thermistor 3[4] : LED-BLUE 3[5] : LED-ORANGE"
- board text removed: "v1.0.0"
